Commit message: Modified urdf to include lidar and resized the camera to make space for lidar

File: eklavya5_description/robots/chasisss.URDF (robot description, URDF)
Before this commit: robot chasisss, 7 links, 6 joints
Links:
- added link hokuyo_link, mass 1e-5; collision box size=0.025 0.025 0.025; visual mesh filename=package://eklavya5_description/meshes/hokuyo.dae
Joints:
- added joint hokuyo_joint: type fixed, parent Steering, child hokuyo_link, origin xyz=0.025 0 0.4 rpy=0 0 0, axis 0 1 0

File: eklavya5_description/robots/chasisss.urdf (robot description, URDF)
Before this commit: robot chasisss, 7 links, 6 joints
Links:
- added link hokuyo_link, mass 1e-5; collision box size=0.025 0.025 0.025; visual mesh filename=package://eklavya5_description/meshes/hokuyo.dae
- link camera_link: geometry collision box size=0.025 0.025 0.025; visual box size=0.025 0.025 0.025
Joints:
- added joint hokuyo_joint: type fixed, parent Steering, child hokuyo_link, origin xyz=0.025 0 0.4 rpy=0 0 0, axis 0 1 0
- joint camera_joint: origin xyz=0.05 0 0.5 rpy=0 0 0 -> xyz=0.025 0 0.5 rpy=0 0 0
