Commit message: Changed Lidar plugin as the previous plugin was not working properly. Removed the repetitive chasisss.URDF

File: eklavya5_description/robots/chasisss.urdf (robot description, URDF)
Before this commit: robot chasisss, 8 links, 7 joints
Joints:
- joint hokuyo_joint: origin xyz=0.025 0 0.4 rpy=0 0 0 -> xyz=0.05 0 0.4 rpy=0 0 0

Commit message: Relocation of sensor position

File: eklavya5_description/robots/chasisss.urdf (robot description, URDF)
Before this commit: robot chasisss, 8 links, 7 joints
Links:
- link camera_link: geometry collision box size=0.05 0.05 0.05; visual box size=0.05 0.05 0.05
Joints:
- joint camera_joint: origin xyz=0.025 0 0.5 rpy=0 0 0 -> xyz=0.05 0 0.5 rpy=0 0 0
- joint hokuyo_joint: origin xyz=0.05 0 0.4 rpy=0 0 0 -> xyz=-0.2 0 0.8 rpy=0 0 0; parent Steering -> base_link
